Commit message: Add Shelf to demo3

File: exercises/Optimization_Based_Planning/solution_ws/src/demo3_support/urdf/demo3.urdf (robot description, URDF)
Before this commit: robot robot, 12 links, 11 joints
Links:
- added link shelf_1; collision box size=0.05 0.5096 1.8288; collision box size=0.05 0.5096 1.8288
Joints:
- added joint shelf_1_joint: type fixed, parent world, child shelf_1, origin xyz=-0.85 0.8 0.12 rpy=0 0 4.7124

File: exercises/Optimization_Based_Planning/solution_ws/src/demo3_support/urdf/environment.xacro (robot description, xacro)
@@ -58,4 +58,61 @@
   </joint>
 </xacro:macro>
+<!-- Shelf -->
+<xacro:macro name="shelf" params="id parent_link *location">
+  <link name="shelf_${id}">
+  <visual>
+    <geometry>
+      <mesh filename="package://demo3_support/meshes/shelf.STL"/>
+    </geometry>
+    <material name="light_gray"/>
+  </visual>
+    <collision name="shelf_${id}_back">
+      <geometry>
+        <box size="0.9144 0.05 1.8288"/>
+      </geometry>
+      <origin xyz="0.4572 0.0 0.9144"/>
+    </collision>
+    <collision name="shelf_${id}_sideL">
+      <geometry>
+        <box size="0.05 0.5096 1.8288"/>
+      </geometry>
+      <origin xyz="0.025 0.22 0.9144"/>
+    </collision>
+    <collision name="shelf_${id}_sideR">
+      <geometry>
+        <box size="0.05 0.5096 1.8288"/>
+      </geometry>
+      <origin xyz=".945 0.22 0.9144"/>
+    </collision>
+    <collision name="shelf_${id}_shelf1">
+      <geometry>
+        <box size="0.9144 0.5096 0.05"/>
+      </geometry>
+      <origin xyz=".4572 0.22 0.025"/>
+    </collision>
+    <collision name="shelf_${id}_shelf2">
+      <geometry>
+        <box size="0.9144 0.5096 0.05"/>
+      </geometry>
+      <origin xyz=".4572 0.22 0.6346"/>
+    </collision>
+    <collision name="shelf_${id}_shelf3">
+      <geometry>
+        <box size="0.9144 0.5096 0.05"/>
+      </geometry>
+      <origin xyz=".4572 0.22 1.2442"/>
+    </collision>
+    <collision name="shelf_${id}_shelf4">
+       <geometry>
+         <box size="0.9144 0.5096 0.05"/>
+       </geometry>
+       <origin xyz=".4572 0.22 1.8038"/>
+    </collision>
+  </link>
+  <joint name="shelf_${id}_joint" type ="fixed">
+    <xacro:insert_block name="location" />
+    <parent link="${parent_link}"/>
+    <child link="shelf_${id}"/>
+  </joint>
 </xacro:macro>
 </robot>

File: exercises/Optimization_Based_Planning/solution_ws/src/demo3_support/urdf/robot.urdf.xacro (robot description, xacro)
@@ -12,8 +12,7 @@
         <origin xyz="0.0 0.0 0.77153" rpy="0 0 0"/>
     </xacro:workcell >
-    <xacro:include filename="$(find demo3_support)/urdf/environment.xacro"/>
-    <xacro:cube parent_link="workcell_base" >
-        <origin xyz="0.15 0.4 0.1" rpy="0 0 0"/>
-    </xacro:cube >
+    <xacro:shelf id="1" parent_link="world" >
+         <origin rpy="0 0 4.7124" xyz="-0.85 0.8 0.12"/>
+    </xacro:shelf >
     <!-- Create joints -->
     <joint name="workcell_base_to_base" type="fixed">

Commit message: Demo3: Move place location to shelf
I also lowered the shelf by 1cm to make it even with the table.

File: exercises/Optimization_Based_Planning/solution_ws/src/demo3_support/urdf/demo3.urdf (robot description, URDF)
Before this commit: robot robot, 13 links, 12 joints
Joints:
- joint shelf_1_joint: origin xyz=-0.85 0.8 0.12 rpy=0 0 4.7124 -> xyz=-0.85 0.8 0.11 rpy=0 0 4.7124

File: exercises/Optimization_Based_Planning/solution_ws/src/demo3_support/urdf/robot.urdf.xacro (robot description, xacro)
@@ -13,5 +13,5 @@
     </xacro:workcell >
     <xacro:shelf id="1" parent_link="world" >
-         <origin rpy="0 0 4.7124" xyz="-0.85 0.8 0.12"/>
+         <origin rpy="0 0 4.7124" xyz="-0.85 0.8 0.11"/>
     </xacro:shelf >
     <!-- Create joints -->
