Commit message: Demo 3: Switch to KUKA iiwa and update workcell STL

File: exercises/Optimization_Based_Planning/solution_ws/src/pick_and_place_support/urdf/pick_and_place.urdf (robot description, URDF)
Before this commit: robot robot, 13 links, 12 joints
Links:
- removed link panda_link0
- removed link panda_link1
- removed link panda_link2
- removed link panda_link3
- removed link panda_link4
- removed link panda_link5
- removed link panda_link6
- removed link panda_link7
- removed link panda_link8
- removed link shelf_1
- added link iiwa_link_0, mass 5; collision mesh filename=package://iiwa_description/meshes/iiwa7/collision/link_0.stl; visual mesh filename=package://iiwa_description/meshes/iiwa7/visual/link_0.stl
- added link iiwa_link_1, mass 3.4525; collision mesh filename=package://iiwa_description/meshes/iiwa7/collision/link_1.stl; visual mesh filename=package://iiwa_description/meshes/iiwa7/visual/link_1.stl
- added link iiwa_link_2, mass 3.4821; collision mesh filename=package://iiwa_description/meshes/iiwa7/collision/link_2.stl; visual mesh filename=package://iiwa_description/meshes/iiwa7/visual/link_2.stl
- added link iiwa_link_3, mass 4.05623; collision mesh filename=package://iiwa_description/meshes/iiwa7/collision/link_3.stl; visual mesh filename=package://iiwa_description/meshes/iiwa7/visual/link_3.stl
- added link iiwa_link_4, mass 3.4822; collision mesh filename=package://iiwa_description/meshes/iiwa7/collision/link_4.stl; visual mesh filename=package://iiwa_description/meshes/iiwa7/visual/link_4.stl
- added link iiwa_link_5, mass 2.1633; collision mesh filename=package://iiwa_description/meshes/iiwa7/collision/link_5.stl; visual mesh filename=package://iiwa_description/meshes/iiwa7/visual/link_5.stl
- added link iiwa_link_6, mass 2.3466; collision mesh filename=package://iiwa_description/meshes/iiwa7/collision/link_6.stl; visual mesh filename=package://iiwa_description/meshes/iiwa7/visual/link_6.stl
- added link iiwa_link_7, mass 3.129; collision mesh filename=package://iiwa_description/meshes/iiwa7/collision/link_7.stl; visual mesh filename=package://iiwa_description/meshes/iiwa7/visual/link_7.stl
- added link iiwa_link_ee
Joints:
- removed joint panda_joint1
- removed joint panda_joint2
- removed joint panda_joint3
- removed joint panda_joint4
- removed joint panda_joint5
- removed joint panda_joint6
- removed joint panda_joint7
- removed joint panda_joint8
- removed joint panda_joint_base_link
- removed joint shelf_1_joint
- added joint base_link_iiwa_joint: type fixed, parent base_link, child iiwa_link_0, origin xyz=0.0 0 0.0 rpy=0 0 0
- added joint iiwa_joint_1: type revolute, parent iiwa_link_0, child iiwa_link_1, origin xyz=0 0 0.15 rpy=0 0 0, axis 0 0 1, limit lower=-2.96705972839 upper=2.96705972839 effort=300 velocity=10
- added joint iiwa_joint_2: type revolute, parent iiwa_link_1, child iiwa_link_2, origin xyz=0 0 0.19 rpy=1.57079632679   0 3.14159265359, axis 0 0 1, limit lower=-2.09439510239 upper=2.09439510239 effort=300 velocity=10
- added joint iiwa_joint_3: type revolute, parent iiwa_link_2, child iiwa_link_3, origin xyz=0 0.21 0 rpy=1.57079632679 0 3.14159265359, axis 0 0 1, limit lower=-2.96705972839 upper=2.96705972839 effort=300 velocity=10
- added joint iiwa_joint_4: type revolute, parent iiwa_link_3, child iiwa_link_4, origin xyz=0 0 0.19 rpy=1.57079632679 0 0, axis 0 0 1, limit lower=-2.09439510239 upper=2.09439510239 effort=300 velocity=10
- added joint iiwa_joint_5: type revolute, parent iiwa_link_4, child iiwa_link_5, origin xyz=0 0.21 0 rpy=-1.57079632679 3.14159265359 0, axis 0 0 1, limit lower=-2.96705972839 upper=2.96705972839 effort=300 velocity=10
- added joint iiwa_joint_6: type revolute, parent iiwa_link_5, child iiwa_link_6, origin xyz=0 0.06070 0.19 rpy=1.57079632679 0 0, axis 0 0 1, limit lower=-2.09439510239 upper=2.09439510239 effort=300 velocity=10
- added joint iiwa_joint_7: type revolute, parent iiwa_link_6, child iiwa_link_7, origin xyz=0 0.081 0.06070 rpy=-1.57079632679 3.14159265359 0, axis 0 0 1, limit lower=-3.05432619099 upper=3.05432619099 effort=300 velocity=10
- added joint iiwa_joint_ee: type fixed, parent iiwa_link_7, child iiwa_link_ee, origin xyz=0 0 0.045 rpy=0 0 0

File: exercises/Optimization_Based_Planning/solution_ws/src/pick_and_place_support/urdf/robot.urdf.xacro (robot description, xacro)
@@ -4,7 +4,12 @@
     <link name="world"/>
     <link name="base_link"/>
+    <!-- Import Rviz colors -->
+    <xacro:include filename="$(find iiwa_description)/urdf/materials.xacro" />
+    <!--Import the lbr iiwa macro -->
+    <xacro:include filename="$(find iiwa_description)/urdf/iiwa7.xacro"/>
     <!-- Include robot -->
-    <xacro:include filename="$(find pick_and_place_support)/urdf/panda_arm.xacro"/>
-    <xacro:panda_arm connected_to="base_link"/>
+    <xacro:iiwa7 hardware_interface="PositionJointInterface" robot_name="iiwa" parent="base_link">
+        <origin xyz="0.0 0 0.0" rpy="0 0 0"/>
+    </xacro:iiwa7>
     <!-- Include workcell (creates joint from world to workcell_base)-->
     <xacro:include filename="$(find pick_and_place_support)/urdf/environment.xacro"/>
@@ -12,7 +17,4 @@
         <origin xyz="0.0 0.0 0.77153" rpy="0 0 0"/>
     </xacro:workcell >
-    <xacro:shelf id="1" parent_link="world" >
-         <origin rpy="0 0 4.7124" xyz="-0.85 0.8 0.11"/>
-    </xacro:shelf >
     <!-- Create joints -->
     <joint name="workcell_base_to_base" type="fixed">
@@ -21,10 +23,3 @@
       <origin xyz="0 0 0.00953" rpy="0 0 1.5708"/>
     </joint>
-    <!--
-    <joint name="base_to_panda_link0" type="fixed">
-      <parent link="base_link"/>
-      <child link="panda_link0"/>
-      <origin xyz="0 0 0" rpy="0 0 0"/>
-    </joint>
--->
 </robot>

Commit message: Demo3: Misc Fixes

File: exercises/Optimization_Based_Planning/solution_ws/src/pick_and_place_support/urdf/pick_and_place.urdf (robot description, URDF)
Before this commit: robot robot, 12 links, 11 joints
Joints:
- joint workcell_base_to_base: origin xyz=0 0 0.00953 rpy=0 0 1.5708 -> xyz=0 -0.0381 0.00953 rpy=0 0 1.5708

File: exercises/Optimization_Based_Planning/solution_ws/src/pick_and_place_support/urdf/robot.urdf.xacro (robot description, xacro)
@@ -21,5 +21,5 @@
       <parent link="workcell_base"/>
       <child link="base_link"/>
-      <origin xyz="0 0 0.00953" rpy="0 0 1.5708"/>
+      <origin xyz="0 -0.0381 0.00953" rpy="0 0 1.5708"/>
     </joint>
 </robot>
