Commit message: Demo3: Add updated cabinet and tune optimization params

File: exercises/Optimization_Based_Planning/solution_ws/src/pick_and_place_support/urdf/environment.xacro (robot description, xacro)
@@ -59,4 +59,19 @@
 </xacro:macro>
 <!-- Shelf -->
+<xacro:macro name="cabinet" params="id parent_link *location">
+  <link name="cabinet_${id}">
+  <collision>
+    <geometry>
+      <mesh filename="package://pick_and_place_support/meshes/cabinet.STL"/>
+    </geometry>
+  </collision>
+  </link>
+<joint name="cabinet_${id}_joint" type ="fixed">
+  <xacro:insert_block name="location" />
+  <parent link="${parent_link}"/>
+  <child link="cabinet_${id}"/>
+</joint>
+</xacro:macro>
+<!-- Shelf -->
 <xacro:macro name="shelf" params="id parent_link *location">
   <link name="shelf_${id}">

File: exercises/Optimization_Based_Planning/solution_ws/src/pick_and_place_support/urdf/pick_and_place.urdf (robot description, URDF)
Before this commit: robot robot, 12 links, 11 joints
Links:
- added link cabinet_1; collision mesh filename=package://pick_and_place_support/meshes/cabinet.STL
Joints:
- added joint cabinet_1_joint: type fixed, parent workcell_base, child cabinet_1, origin xyz=-0.3048 1.016 0.771525 rpy=0 0 0

File: exercises/Optimization_Based_Planning/solution_ws/src/pick_and_place_support/urdf/robot.urdf.xacro (robot description, xacro)
@@ -17,4 +17,7 @@
         <origin xyz="0.0 0.0 0.77153" rpy="0 0 0"/>
     </xacro:workcell >
+    <xacro:cabinet id="1" parent_link="workcell_base" >
+        <origin rpy="0 0 0" xyz="-0.3048 1.016 0.771525"/>
+    </xacro:cabinet >
     <!-- Create joints -->
     <joint name="workcell_base_to_base" type="fixed">

Commit message: Fix collision
Had a nonconvex mesh as the collision model for the shelf. Replaced with convex shapes.

File: exercises/Optimization_Based_Planning/solution_ws/src/pick_and_place_support/urdf/environment.xacro (robot description, xacro)
@@ -58,12 +58,49 @@
   </joint>
 </xacro:macro>
-<!-- Shelf -->
+<!-- cabinet - Visual is in workcell_base.stl-->
 <xacro:macro name="cabinet" params="id parent_link *location">
   <link name="cabinet_${id}">
-  <collision>
+<collision name="cabinet_${id}_back">
+  <geometry>
+    <box size="0.5969 0.0254 0.762"/>
+  </geometry>
+  <origin xyz=".2985 -.0127 -0.381"/>
+</collision>
+<collision name="cabinet_${id}_sideL">
+  <geometry>
+    <box size="0.0254 0.3048 0.762"/>
+  </geometry>
+  <origin xyz="0.0127 -0.1524 -0.381"/>
+</collision>
+<collision name="cabinet_${id}_sideR">
+<geometry>
+  <box size="0.0254 0.3048 0.762"/>
+</geometry>
+<origin xyz="0.5969 -0.1524 -0.381"/>
+</collision>
+<collision name="cabinet_${id}_cabinet1">
+     <geometry>
+          <box size="0.5969 0.3048 0.0254"/>
+    </geometry>
+    <origin xyz=".2985 -0.1524  -0.7493"/>
+</collision>
+<collision name="cabinet_${id}_cabinet2">
     <geometry>
-      <mesh filename="package://pick_and_place_support/meshes/cabinet.STL"/>
+        <box size="0.5969 0.3048 0.0254"/>
     </geometry>
-  </collision>
+    <origin xyz=".2985 -0.1524  -0.508"/>
+</collision>
+<collision name="cabinet_${id}_cabinet3">
+    <geometry>
+        <box size="0.5969 0.3048 0.0254"/>
+    </geometry>
+    <origin xyz=".2985 -0.1524  -0.254"/>
+</collision>
+<collision name="cabinet_${id}_cabinet4">
+    <geometry>
+        <box size="0.5969 0.3048 0.0254"/>
+    </geometry>
+    <origin xyz=".2985 -0.1524  -0.0127"/>
+</collision>
   </link>
 <joint name="cabinet_${id}_joint" type ="fixed">
@@ -73,5 +110,5 @@
 </joint>
 </xacro:macro>
-<!-- Shelf -->
+<!-- Shelf - Not currently used-->
 <xacro:macro name="shelf" params="id parent_link *location">
   <link name="shelf_${id}">

File: exercises/Optimization_Based_Planning/solution_ws/src/pick_and_place_support/urdf/pick_and_place.urdf (robot description, URDF)
Before this commit: robot robot, 13 links, 12 joints
Links:
- link cabinet_1: geometry collision box size=0.0254 0.3048 0.762; collision box size=0.0254 0.3048 0.762
