Commit message: Demo 3: Update template to match solution

File: exercises/Optimization_Based_Planning/template_ws/src/pick_and_place_support/urdf/environment.xacro (robot description, xacro)
@@ -59,4 +59,19 @@
 </xacro:macro>
 <!-- Shelf -->
+<xacro:macro name="cabinet" params="id parent_link *location">
+  <link name="cabinet_${id}">
+  <collision>
+    <geometry>
+      <mesh filename="package://pick_and_place_support/meshes/cabinet.STL"/>
+    </geometry>
+  </collision>
+  </link>
+<joint name="cabinet_${id}_joint" type ="fixed">
+  <xacro:insert_block name="location" />
+  <parent link="${parent_link}"/>
+  <child link="cabinet_${id}"/>
+</joint>
+</xacro:macro>
+<!-- Shelf -->
 <xacro:macro name="shelf" params="id parent_link *location">
   <link name="shelf_${id}">

File: exercises/Optimization_Based_Planning/template_ws/src/pick_and_place_support/urdf/pick_and_place.urdf (robot description, URDF)
Before this commit: robot robot, 12 links, 11 joints
Links:
- added link cabinet_1; collision mesh filename=package://pick_and_place_support/meshes/cabinet.STL
Joints:
- added joint cabinet_1_joint: type fixed, parent workcell_base, child cabinet_1, origin xyz=-0.3048 1.016 0.771525 rpy=0 0 0
- joint workcell_base_to_base: origin xyz=0 0 0.00953 rpy=0 0 1.5708 -> xyz=0 -0.0381 0.00953 rpy=0 0 1.5708

File: exercises/Optimization_Based_Planning/template_ws/src/pick_and_place_support/urdf/robot.urdf.xacro (robot description, xacro)
@@ -17,9 +17,12 @@
         <origin xyz="0.0 0.0 0.77153" rpy="0 0 0"/>
     </xacro:workcell >
+    <xacro:cabinet id="1" parent_link="workcell_base" >
+        <origin rpy="0 0 0" xyz="-0.3048 1.016 0.771525"/>
+    </xacro:cabinet >
     <!-- Create joints -->
     <joint name="workcell_base_to_base" type="fixed">
       <parent link="workcell_base"/>
       <child link="base_link"/>
-      <origin xyz="0 0 0.00953" rpy="0 0 1.5708"/>
+      <origin xyz="0 -0.0381 0.00953" rpy="0 0 1.5708"/>
     </joint>
 </robot>
